File: Smart_Grid_Prototype/PCB/new kicad.kicad_pcb (KiCad board)
At the start: 2 copper layers, 144.8 x 116.8 mm, 70 parts, among them J1 EXT_POW, J2 24VAC _LOAD, J3 AC_INPUT, J4 DC_LOAD, J5 POW_SHARE, Q1 BD139, Q2 BD139, Q3 BD139, Q4 BD139, Q5 BD139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

Commit message: pcb updated with accrate component names
Parts:
- D1: value 1N5408/RELAY_FWD -> 1N5408/DIODE
- D2: value 1N5408/RELAY-1_FWD -> 1N5408/DIODE
- D3: value GBU4A -> GBU4A/BRIDGE_RECT
- D7: value LOAD_INDICATOR -> LOAD_STATUS
- R11, R2, R4, R5, R6, R7, R9: value 220 -> 220R
- R14: value 1.5kR -> 1.5k
- R15: value 2kR -> 2k
- R23, R24, R26, R3, R31: value 1 -> 1R
- R27: value 150 -> 150R
- U1: value ZC563900 -> ESP8266
- U10, U6: value MODERATE_V -> PC817
- U11: value HIGH_V -> PC817
- U2: value CKT_1_POWER_CON -> RELAY_INT
- U3: value CKT_1_POWER_CON -> RELAY_PS
- U4, U9: value MIN_V -> PC817
Other:
- board text added: "+"
- board text added: "-"
- board text added: "DC_LOAD"
- board text added: "EXT_POWER"
- board text added: "POW_READY"
- board text added: "POW_SHARE"
- board text added: "POW_STATUS"
- board text added: "POW_STATUS_2"
- board text added: "~"
Changed lines of the file:
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@@
 			(psa4output no)
 			(plotreference yes)
-			(plotvalue no)
+			(plotvalue yes)
 			(plotfptext yes)
 			(plotinvisibletext no)
@@
 			(drillshape 0)
 			(scaleselection 1)
-			(outputdirectory "KiCad agerber/PCB with ccet logo/")
+			(outputdirectory "gerber_to_order/")
 		)
 	)
@@
 			)
 		)
-		(property "Value" "ZC563900"
+		(property "Value" "ESP8266"
 			(at 1.27 19.812 0)
 			(layer "F.Fab")
@@
 			)
 		)
-		(property "Value" "MIN_V"
+		(property "Value" "PC817"
 			(at 3.81 4.87 0)
 			(layer "F.Fab")
@@
 			)
 		)
-		(property "Value" "220"
+		(property "Value" "220R"
 			(at 7.62 2.37 90)
 			(layer "F.Fab")
@@
 			)
 		)
-		(property "Value" "1"
+		(property "Value" "1R"
 			(at 15.24 4.32 0)
 			(layer "F.Fab")
@@
 			)
 		)
-		(property "Value" "220"
+		(property "Value" "220R"
 			(at 7.62 2.37 0)
 			(layer "F.Fab")
@@
 			)
 		)
-		(property "Value" "GBU4A"
+		(property "Value" "GBU4A/BRIDGE_RECT"
 			(at 7.1 -2.5 90)
 			(layer "F.Fab")
@@
 			)
 		)
-		(property "Value" "1.5kR"
+		(property "Value" "1.5k"
 			(at 7.62 2.37 90)
 			(layer "F.Fab")
@@
 			)
 		)
-		(property "Value" "150"
+		(property "Value" "150R"
 			(at 7.62 2.37 90)
 			(layer "F.Fab")
@@
 			)
 		)
-		(property "Value" "1"
+		(property "Value" "1R"
 			(at 12.7 4.12 90)
 			(layer "F.Fab")
@@
 			)
 		)
-		(property "Value" "220"
+		(property "Value" "220R"
 			(at 7.62 2.37 0)
 			(layer "F.Fab")
@@
 			)
 		)
-		(property "Value" "220"
+		(property "Value" "220R"
 			(at 7.62 2.37 90)
 			(layer "F.Fab")
@@
 			)
 		)
-		(property "Value" "1"
+		(property "Value" "1R"
 			(at 15.24 4.32 90)
 			(layer "F.Fab")
@@
 			)
 		)
-		(property "Value" "220"
+		(property "Value" "220R"
 			(at 7.62 2.37 90)
 			(layer "F.Fab")
@@
 			)
 		)
-		(property "Value" "HIGH_V"
+		(property "Value" "PC817"
 			(at 3.81 4.87 0)
 			(layer "F.Fab")
@@
 			)
 		)
-		(property "Value" "220"
+		(property "Value" "220R"
 			(at 7.62 2.37 90)
 			(layer "F.Fab")
@@
 			)
 		)
-		(property "Value" "220"
+		(property "Value" "220R"
 			(at 7.62 2.37 0)
 			(layer "F.Fab")
@@
 			)
 		)
-		(property "Value" "2kR"
+		(property "Value" "2k"
 			(at 7.62 2.37 0)
 			(layer "F.Fab")
@@
 			)
 		)
-		(property "Value" "CKT_1_POWER_CON"
+		(property "Value" "RELAY_INT"
 			(at 22.10675 -10.21175 90)
 			(layer "F.SilkS")
@@
 			)
 		)
-		(property "Value" "CKT_1_POWER_CON"
+		(property "Value" "RELAY_PS"
 			(at 9.40675 -10.21175 0)
 			(layer "F.SilkS")
@@
 			)
 		)
-		(property "Value" "LOAD_INDICATOR"
+		(property "Value" "LOAD_STATUS"
 			(at 1.27 3.96 0)
 			(layer "F.Fab")
@@
 			)
 		)
-		(property "Value" "1N5408/RELAY_FWD"
+		(property "Value" "1N5408/DIODE"
 			(at 6.35 2.97 90)
 			(layer "F.Fab")
@@
 			)
 		)
-		(property "Value" "1"
+		(property "Value" "1R"
 			(at 15.24 4.32 90)
 			(layer "F.Fab")
@@
 			)
 		)
-		(property "Value" "MIN_V"
+		(property "Value" "PC817"
 			(at 3.81 4.87 90)
 			(layer "F.Fab")
@@
 			)
 		)
-		(property "Value" "MODERATE_V"
+		(property "Value" "PC817"
 			(at 3.81 4.87 0)
 			(layer "F.Fab")
@@
 			)
 		)
-		(property "Value" "1"
+		(property "Value" "1R"
 			(at 15.24 4.32 90)
 			(layer "F.Fab")
@@
 			)
 		)
-		(property "Value" "MODERATE_V"
+		(property "Value" "PC817"
 			(at 3.81 4.87 0)
 			(layer "F.Fab")
@@
 			)
 		)
-		(property "Value" "1N5408/RELAY-1_FWD"
+		(property "Value" "1N5408/DIODE"
 			(at 6.35 2.97 90)
 			(layer "F.Fab")
@@
 		(layer "Edge.Cuts")
 	)
+	(gr_text "DC_LOAD\n"
+		(at 116.84 149.86 0)
+		(layer "F.SilkS")
+		(effects
+			(font
+				(size 0.8 0.7)
+				(thickness 0.1)
+			)
+			(justify left bottom)
+		)
+	)
 	(gr_text "SMART GRID PROTOTYPE"
 		(at 78.74 45.72 0)
@@
 		)
 	)
+	(gr_text "~\n"
+		(at 213.36 86.36 90)
+		(layer "F.SilkS")
+		(effects
+			(font
+				(size 1 1.5)
+				(thickness 0.1)
+			)
+			(justify left bottom)
+		)
+	)
+	(gr_text "~\n"
+		(at 213.36 111.76 90)
+		(layer "F.SilkS")
+		(effects
+			(font
+				(size 1 1.5)
+				(thickness 0.1)
+			)
+			(justify left bottom)
+		)
+	)
+	(gr_text "POW_STATUS_2\n"
+		(at 177.8 116.84 90)
+		(layer "F.SilkS")
+		(effects
+			(font
+				(size 0.8 0.7)
+				(thickness 0.1)
+			)
+			(justify left bottom)
+		)
+	)
+	(gr_text "-"
+		(at 154.94 149.86 0)
+		(layer "F.SilkS")
+		(effects
+			(font
+				(size 1.6 1.6)
+				(thickness 0.1)
+			)
+			(justify left bottom)
+		)
+	)
+	(gr_text "-"
+		(at 213.36 149.86 0)
+		(layer "F.SilkS")
+		(effects
+			(font
+				(size 1.6 1.6)
+				(thickness 0.1)
+			)
+			(justify left bottom)
+		)
+	)
+	(gr_text "POW_READY\n"
+		(at 177.8 124.46 90)
+		(layer "F.SilkS")
+		(effects
+			(font
+				(size 0.8 0.7)
+				(thickness 0.1)
+			)
+			(justify left bottom)
+		)
+	)
+	(gr_text "+"
+		(at 200.66 149.86 0)
+		(layer "F.SilkS")
+		(effects
+			(font
+				(size 1.5 1.5)
+				(thickness 0.1)
+			)
+			(justify left bottom)
+		)
+	)
+	(gr_text "-"
+		(at 124.46 149.86 0)
+		(layer "F.SilkS")
+		(effects
+			(font
+				(size 1.6 1.6)
+				(thickness 0.1)
+			)
+			(justify left bottom)
+		)
+	)
+	(gr_text "~\n"
+		(at 213.36 119.38 90)
+		(layer "F.SilkS")
+		(effects
+			(font
+				(size 1 1.5)
+				(thickness 0.1)
+			)
+			(justify left bottom)
+		)
+	)
 	(gr_text "MCO21576 RAJEEV KHARE\nMCO21578 SOHAM JAISWAL\nLCO21585 ANKUSH VERMA"
 		(at 83.82 58.42 0)
@@
 		)
 	)
+	(gr_text "POW_SHARE\n"
+		(at 205.74 149.86 0)
+		(layer "F.SilkS")
+		(effects
+			(font
+				(size 0.8 0.7)
+				(thickness 0.1)
+			)
+			(justify left bottom)
+		)
+	)
+	(gr_text "POW_STATUS\n"
+		(at 177.8 106.68 90)
+		(layer "F.SilkS")
+		(effects
+			(font
+				(size 0.8 0.7)
+				(thickness 0.1)
+			)
+			(justify left bottom)
+		)
+	)
+	(gr_text "EXT_POWER\n"
+		(at 160.02 149.86 0)
+		(layer "F.SilkS")
+		(effects
+			(font
+				(size 0.8 0.7)
+				(thickness 0.1)
+			)
+			(justify left bottom)
+		)
+	)
+	(gr_text "+"
+		(at 167.64 149.86 0)
+		(layer "F.SilkS")
+		(effects
+			(font
+				(size 1.5 1.5)
+				(thickness 0.1)
+			)
+			(justify left bottom)
+		)
+	)
+	(gr_text "+"
+		(at 114.3 149.86 0)
+		(layer "F.SilkS")
+		(effects
+			(font
+				(size 1.5 1.5)
+				(thickness 0.1)
+			)
+			(justify left bottom)
+		)
+	)
+	(gr_text "~\n"
+		(at 213.36 81.28 90)
+		(layer "F.SilkS")
+		(effects
+			(font
+				(size 1 1.5)
+				(thickness 0.1)
+			)
+			(justify left bottom)
+		)
+	)
