File: Smart_Grid_Prototype/Schematic/new kicad.kicad_sch (KiCad schematic)
At the start: 70 parts, among them J1 EXT_POW, J2 24VAC _LOAD, J3 AC_INPUT, J4 DC_LOAD, J5 POW_SHARE, Q1 BD139, Q2 BD139, Q3 BD139, Q4 BD139, Q5 BD139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

Commit message: pcb and schematic updated
Connections:
- net EXT_POWER: now also U1.15 (VIN)
- no-connect marks 14 -> 13
Changed lines of the file:
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@@
-	)
-	(no_connect
-		(at 17.78 146.05)
 	)
 	(no_connect
@@
 		(fields_autoplaced yes)
 		(effects
+			(font
+				(size 1.27 1.27)
+			)
+			(justify left bottom)
+		)
+	)
+	(label "EXT_POWER"
+		(at 17.78 146.05 0)
+		(fields_autoplaced yes)
+		(effects
