File: Smart_Grid_Prototype/Schematic/new kicad.kicad_pcb (KiCad board)
At the start: 2 copper layers, 144.8 x 116.8 mm, 70 parts, among them J1 EXT_POW, J2 24VAC _LOAD, J3 AC_INPUT, J4 DC_LOAD, J5 POW_SHARE, Q1 BD139, Q2 BD139, Q3 BD139, Q4 BD139, Q5 BD139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

Commit message: pcb and schematic updated
Connections:
- U1 pad 15: unconnected-(U1-VIN-Pad15) -> /EXT_POWER
Routing:
- net GND: track 452.7 -> 514.2 mm
- net /EXT_POWER: track 114.2 -> 162.5 mm
- added copper zone on B.Cu, net (none)
- added copper zone on F.Cu, net (none)
- removed copper zone on B.Cu, net GND
- removed copper zone on F.Cu, net GND

Commit message: only saved
Routing:
- added copper zone on B.Cu, net GND
- added copper zone on F.Cu, net GND
- removed copper zone on B.Cu, net (none)
- removed copper zone on F.Cu, net (none)
Changed lines of the file:
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@@
 	)
 	(zone
-		(net 0)
-		(net_name "")
+		(net 1)
+		(net_name "GND")
 		(layers "F&B.Cu")
 		(hatch edge 0.5)
@@
 			(thermal_gap 0.5)
 			(thermal_bridge_width 0.5)
-			(island_removal_mode 1)
-			(island_area_min 10)
 		)
 		(polygon
 			(pts
-				(xy 68.58 152.4) (xy 76.2 160.02) (xy 220.98 160.02) (xy 226.06 154.94) (xy 226.06 33.02) (xy 68.58 33.02)
+				(xy 68.58 33.02) (xy 68.58 154.94) (xy 218.44 154.94) (xy 218.44 33.02)
 			)
 		)
