File: Smart_Grid_Prototype/Schematic+PCB+GRBR/new kicad.kicad_pcb (KiCad board)
At the start: 2 copper layers, 148.5 x 117.2 mm, 78 parts, among them J1 EXT_POW, J2 AC_LOAD, J3 AC_STEPDOWN, J4 DC_LOAD, J5 POW_SHARE, J6 USB_C_Receptacle_PowerOnly_6P, J7 220VAC, J8 220VAC-TRANS, K1 G3MB-202PDC5, Q1 BD139, Q2 BD139, Q3 BD139, Q4 BD139, Q5 BD139, Q6 BD139, Q7 BD139, Q8 BD139, U1 ESP8266, U10 PC817, U11 PC817, U12 PC817, U13 PC817, U14 PC817, U15 PC817, U16 PC817, U2 RELAY_INT, U3 RELAY_PS, U4 PC817, U5 LM7824_TO220, U6 PC817, U7 PC817, U8 LM317_TO-220, U9 PC817

Commit message: header pin added
Parts:
- added J9: Conn_01x06_Socket, Connector_PinHeader_2.54mm:PinHeader_1x06_P2.54mm_Vertical, F.Cu at (74.0, 89.7)
Connections:
- U1 pad 4: unconnected-(U1-SD3-Pad4) -> /SD3
- U1 pad 5: unconnected-(U1-SD2-Pad5) -> /SD2
- U1 pad 6: unconnected-(U1-SD1-Pad6) -> /SD1
- U1 pad 7: unconnected-(U1-CMD-Pad7) -> /SD0
- U1 pad 8: unconnected-(U1-SD0-Pad8) -> /CMD
- U1 pad 9: unconnected-(U1-CLK-Pad9) -> /CLK
Routing:
- net /CMD: track 0.00 -> 18.7 mm
- net /SD3: track 0.00 -> 17.7 mm
- net /SD2: track 0.00 -> 17.7 mm
- net /SD1: track 0.00 -> 17.7 mm
- net /SD0: track 0.00 -> 17.7 mm
- net /CLK: track 0.00 -> 17.7 mm
- net GND: vias 34 -> 54
