File: Smart_Grid_Prototype/Schematic+PCB+GRBR/new kicad.kicad_sch (KiCad schematic)
At the start: 78 parts, among them J1 EXT_POW, J2 AC_LOAD, J3 AC_STEPDOWN, J4 DC_LOAD, J5 POW_SHARE, J6 USB_C_Receptacle_PowerOnly_6P, J7 220VAC, J8 220VAC-TRANS, K1 G3MB-202PDC5, Q1 BD139, Q2 BD139, Q3 BD139, Q4 BD139, Q5 BD139, Q6 BD139, Q7 BD139, Q8 BD139, U1 ESP8266, U10 PC817, U11 PC817, U12 PC817, U13 PC817, U14 PC817, U15 PC817, U16 PC817, U2 RELAY_INT, U3 RELAY_PS, U4 PC817, U5 LM7824_TO220, U6 PC817, U7 PC817, U8 LM317_TO-220, U9 PC817

Commit message: header pin added
Parts:
- added J9: Conn_01x06_Socket, Connector_PinHeader_2.54mm:PinHeader_1x06_P2.54mm_Vertical, symbol Connector:Conn_01x06_Socket
Connections:
- net SD3: now reaches U1.4 (SD3)
- net SD3: now also J9.1 (Pin_1)
- net SD2: now reaches U1.5 (SD2)
- net SD2: now also J9.2 (Pin_2)
- net SD1: now reaches U1.6 (SD1)
- net SD1: now also J9.3 (Pin_3)
- net SD0: now reaches U1.7 (CMD)
- net SD0: now also J9.4 (Pin_4)
- net CMD: now reaches U1.8 (SD0)
- net CMD: now also J9.5 (Pin_5)
- net CLK: now reaches U1.9 (CLK)
- net CLK: now also J9.6 (Pin_6)
- no-connect marks 13 -> 7
Other:
- moved on the sheet: C4, R8

Commit message: Esp32,Sdcard initialized,heart sensor project completed--Project
Parts:
- R13: value 500R -> 1.8k
- R14: value 1.5k -> 2.2k
- R15: value 2k -> 800R
- R27: value 150R -> 2k
- R30: value 5k -> 1R
Changed lines of the file:
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@@
 		(dnp no)
 		(property "Reference" "D2"
-			(at 144.78 105.41 0)
+			(at 142.24 107.95 0)
 			(effects
 				(font
@@
 			)
 		)
-		(property "Value" "2k"
+		(property "Value" "800R"
 			(at 264.16 175.26 90)
 			(effects
@@
 			)
 		)
-		(property "Value" "150R"
+		(property "Value" "2k"
 			(at 353.06 138.684 0)
 			(effects
@@
 			)
 		)
-		(property "Value" "1.5k"
+		(property "Value" "2.2k"
 			(at 264.16 161.29 90)
 			(effects
@@
 			)
 		)
-		(property "Value" "5k"
+		(property "Value" "1R"
 			(at 353.06 164.084 0)
 			(effects
@@
 			)
 		)
-		(property "Value" "500R"
+		(property "Value" "1.8k"
 			(at 264.16 134.62 90)
 			(effects
