File: Arduino_UNO_R3/arduino_uno_r3/arduino_uno_r3.kicad_pcb (KiCad board)
At the start: 4 copper layers, 105.4 x 57.5 mm, 58 parts, among them J1 Barrel_Jack_Switch_Pin3Ring, J2 Conn_01x09_Socket, J3 USB-B-S-X-X-TH-TR, J4 ICSP HEADER, J5 Conn_01x04_Socket, J6 ICSP HEADER, J7 Conn_01x08_Socket, J8 Conn_01x10_Socket, J9 Conn_01x06_Socket, Q1 FDN340P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

Commit message: arduino created
Routing:
- net GND: vias 9 -> 45
