File: Arduino_UNO_R3/arduino_uno_r3/MCU.kicad_sch (KiCad schematic)
At the start: 17 parts, among them J6 ICSP HEADER, J7 Conn_01x08_Socket, J8 Conn_01x10_Socket, J9 Conn_01x06_Socket, U6 LMV358, U7 ATMEGA328P-PU, Y2 CSTCE16M0V53-R0

Commit message: arduino created
Parts:
- J6: footprint Library:SAMTEC_TSS-103-03-L-D -> Connector_PinHeader_1.27mm:PinHeader_2x03_P1.27mm_Vertical
Changed lines of the file:
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@@
 			)
 		)
-		(property "Footprint" "Library:SAMTEC_TSS-103-03-L-D"
+		(property "Footprint" "Connector_PinHeader_1.27mm:PinHeader_2x03_P1.27mm_Vertical"
 			(at 110.998 124.968 0)
 			(effects
@@
 				)
 				(justify bottom)
-				(hide yes)
 			)
 		)

Commit message: dont know updates
Parts:
- removed C10, C9: 100n, Capacitor_SMD:CP_Elec_6.3x3, symbol Device:C_Polarized
- removed D6: LED, LED_SMD:LED_0603_1608Metric, symbol Device:LED
- removed D7: D, Diode_SMD:D_0603_1608Metric, symbol Device:D
- removed J6: ICSP HEADER, Connector_PinHeader_1.27mm:PinHeader_2x03_P1.27mm_Vertical, symbol New_Library_0:ICSP HEADER
- removed J7: Conn_01x08_Socket, Connector_Samtec_HPM_THT:Samtec_HPM-08-01-x-S_Straight_1x08_Pitch5.08mm, symbol Connector:Conn_01x08_Socket
- removed J8: Conn_01x10_Socket, Connector_Samtec_HPM_THT:Samtec_HPM-10-01-x-S_Straight_1x10_Pitch5.08mm, symbol Connector:Conn_01x10_Socket
- removed J9: Conn_01x06_Socket, Connector_Samtec_HPM_THT:Samtec_HPM-06-01-x-S_Straight_1x06_Pitch5.08mm, symbol Connector:Conn_01x06_Socket
- removed R12, R15, R16: 1k, Resistor_SMD:R_0603_1608Metric, symbol Device:R
- removed R13: 1M, Resistor_SMD:R_0603_1608Metric, symbol Device:R
- removed R14: 10k, Resistor_SMD:R_0603_1608Metric, symbol Device:R
- removed S1: TL3305CF160QG, Library:SW_TL3305CF160QG, symbol New_Library_0:TL3305CF160QG
- removed U6: LMV358, Library:TO229P990X238-3N, symbol Amplifier_Operational:LM358
- removed U7: ATMEGA328P-PU, Library:DIP794W46P254L2967H457Q28B, symbol New_Library_0:ATMEGA328P-PU
- removed Y2: CSTCE16M0V53-R0, Library:OSC_CSTCE16M0V53-R0, symbol New_Library_0:CSTCE16M0V53-R0
- added C10, C9: 22pf, Capacitor_SMD:C_0805_2012Metric_Pad1.18x1.45mm_HandSolder, symbol Device:C
- added C7, C8: 0.1uf, Capacitor_SMD:C_0805_2012Metric_Pad1.18x1.45mm_HandSolder, symbol Device:C
- added D17: LED, LED_SMD:LED_0805_2012Metric_Pad1.15x1.40mm_HandSolder, symbol Device:LED
- added J10: LCD, Connector_JST:JST_PH_B3B-PH-K_1x03_P2.00mm_Vertical, symbol Connector:Conn_01x03_Pin
- added J14: MOTOR_1, Connector_JST:JST_PH_B2B-PH-K_1x02_P2.00mm_Vertical, symbol Connector:Conn_01x02_Pin
- added J16: IR, Connector_JST:JST_PH_B2B-PH-K_1x02_P2.00mm_Vertical, symbol Connector:Conn_01x02_Pin
- added J18: LED_MATRIX, Connector_JST:JST_PH_B9B-PH-K_1x09_P2.00mm_Vertical, symbol Connector:Conn_01x09_Pin
- added J19: 7 Segment, Connector_JST:JST_PH_B9B-PH-K_1x09_P2.00mm_Vertical, symbol Connector:Conn_01x09_Pin
- added J20: Buzzer, Connector_JST:JST_PH_B2B-PH-K_1x02_P2.00mm_Vertical, symbol Connector:Conn_01x02_Pin
- added J21: RBG_LED, Connector_JST:JST_PH_B3B-PH-K_1x03_P2.00mm_Vertical, symbol Connector:Conn_01x03_Socket
- added J22: US, Connector_JST:JST_PH_B3B-PH-K_1x03_P2.00mm_Vertical, symbol Connector:Conn_01x03_Socket
- added J23: Conn_01x14, Connector_PinHeader_2.54mm:PinHeader_1x14_P2.54mm_Vertical, symbol Connector_Generic:Conn_01x14
- added J24: Potentiometer control, Connector_JST:JST_PH_B2B-PH-K_1x02_P2.00mm_Vertical, symbol Connector:Conn_01x02_Pin
- added J25: PULL DOWN_UP, Connector_JST:JST_PH_B3B-PH-K_1x03_P2.00mm_Vertical, symbol Connector:Conn_01x03_Pin
- added J26: LDR, Connector_JST:JST_PH_B2B-PH-K_1x02_P2.00mm_Vertical, symbol Connector:Conn_01x02_Pin
- added J28: Servo, Connector_JST:JST_PH_B2B-PH-K_1x02_P2.00mm_Vertical, symbol Connector:Conn_01x02_Pin
- added J30: MIC, Connector_JST:JST_PH_B2B-PH-K_1x02_P2.00mm_Vertical, symbol Connector:Conn_01x02_Pin
- added J38: MOTOR_2, Connector_JST:JST_PH_B2B-PH-K_1x02_P2.00mm_Vertical, symbol Connector:Conn_01x02_Pin
- added J39, J40: Conn_01x06, Connector_PinHeader_2.54mm:PinHeader_1x06_P2.54mm_Vertical, symbol Connector_Generic:Conn_01x06
- added R33: 10k, Resistor_SMD:R_0805_2012Metric_Pad1.20x1.40mm_HandSolder, symbol Device:R
- added R34: 4.7k, Resistor_SMD:R_0805_2012Metric_Pad1.20x1.40mm_HandSolder, symbol Device:R
- added SW3: SW_Push, Button_Switch_THT:SW_PUSH_6mm_H4.3mm, symbol Switch:SW_Push
- added U7: ATmega328-A, Package_QFP:TQFP-32_7x7mm_P0.8mm, symbol MCU_Microchip_ATmega:ATmega328-A
- added Y1: Crystal, Crystal:Crystal_SMD_HC49-SD, symbol Device:Crystal
Connections:
- net +5V: now also C8.1, J10.1 (Pin_1), J20.1 (Pin_1), J22.1 (Pin_1), J24.1 (Pin_1), J25.1 (Pin_1), J26.1 (Pin_1), J28.2 (Pin_2), J40.1 (Pin_1), J40.2 (Pin_2), R33.1, U7.18 (AVCC), U7.4 (VCC), U7.6 (VCC)
- net GND: now also C10.2, C7.2, C8.2, C9.2, D17.1 (K), J40.3 (Pin_3), J40.4 (Pin_4), J40.5 (Pin_5), J40.6 (Pin_6), SW3.1, U7.21 (GND), U7.3 (GND), U7.5 (GND)
- net PB5/SCK: now also J23.14 (Pin_14), J25.2 (Pin_2), R34.1, U7.17 (PB5)
- net PC4/SDA: now also J10.2 (Pin_2), J39.5 (Pin_5), U7.27 (PC4)
- net PC5/SCL: now also J10.3 (Pin_3), J39.6 (Pin_6), U7.28 (PC5)
- net RXM8: now also J23.1 (Pin_1), U7.30 (PD0)
- net TXM8: now also J23.2 (Pin_2), U7.31 (PD1)
- new net: C7.1, U7.20 (AREF)
- new net: D17.2 (A), R34.2
- new net: C10.1, U7.8 (XTAL2/PB7), Y1.1
- new net: C9.1, U7.7 (XTAL1/PB6), Y1.2
- new net A0: J30.1 (Pin_1), J39.1 (Pin_1), U7.23 (PC0)
- new net A1: J26.2 (Pin_2), J39.2 (Pin_2), U7.24 (PC1)
- new net A2: J16.1 (Pin_1), J24.2 (Pin_2), J39.3 (Pin_3), U7.25 (PC2)
- new net A3: J16.2 (Pin_2), J39.4 (Pin_4), U7.26 (PC3)
- new net ADC6: U7.19 (ADC6)
- new net ADC7: U7.22 (ADC7)
- new net PB0: J18.7 (Pin_7), J19.7 (Pin_7), J22.3 (Pin_3), J23.9 (Pin_9), U7.12 (PB0)
- new net PB1: J18.8 (Pin_8), J19.8 (Pin_8), J21.1 (Pin_1), J23.10 (Pin_10), J28.1 (Pin_1), U7.13 (PB1)
- new net PB2: J18.9 (Pin_9), J19.9 (Pin_9), J21.2 (Pin_2), J23.11 (Pin_11), J38.1 (Pin_1), U7.14 (PB2)
- new net PB3: J21.3 (Pin_3), J23.12 (Pin_12), J38.2 (Pin_2), U7.15 (PB3)
- new net PB4: J23.13 (Pin_13), J25.3 (Pin_3), U7.16 (PB4)
- new net PC6/~{RESET}: R33.2, SW3.2, U7.29 (~{RESET}/PC6)
- new net PD2: J18.1 (Pin_1), J19.1 (Pin_1), J20.2 (Pin_2), J23.3 (Pin_3), J30.2 (Pin_2), U7.32 (PD2)
- new net PD3: J18.2 (Pin_2), J19.2 (Pin_2), J23.4 (Pin_4), U7.1 (PD3)
- new net PD4: J18.3 (Pin_3), J19.3 (Pin_3), J23.5 (Pin_5), U7.2 (PD4)
- new net PD5: J14.1 (Pin_1), J18.4 (Pin_4), J19.4 (Pin_4), J23.6 (Pin_6), U7.9 (PD5)
- new net PD6: J14.2 (Pin_2), J18.5 (Pin_5), J19.5 (Pin_5), J23.7 (Pin_7), U7.10 (PD6)
- new net PD7: J18.6 (Pin_6), J19.6 (Pin_6), J22.2 (Pin_2), J23.8 (Pin_8), U7.11 (PD7)
- no-connect marks 0 -> 2
Other:
- note added: "8 9 10 11 12 13"
- note added: "Arduino Control Pins"
- note added: "Atmega328-Au"
- note added: "Connectors"
- note added: "IR-A4,A5"
