File: Arduino_UNO_R3/arduino_uno_r3/PWR SEC.kicad_sch (KiCad schematic)
At the start: 18 parts, among them J1 Barrel_Jack_Switch_Pin3Ring, J2 Conn_01x09_Socket, Q1 FDN340P, U1 NCP1117-5.0_TO252, U3 LP2985-3.3, U6 LMV358

Commit message: dont know updates
Parts:
- removed C4: 100n, Capacitor_SMD:CP_Elec_6.3x3, symbol Device:C_Polarized
- removed C5: 1u, Capacitor_SMD:CP_Elec_6.3x3, symbol Device:C_Polarized
- removed J1: Barrel_Jack_Switch_Pin3Ring, Connector_BarrelJack:BarrelJack_Horizontal, symbol Connector:Barrel_Jack_Switch_Pin3Ring
- removed J2: Conn_01x09_Socket, Connector_Samtec_HPM_THT:Samtec_HPM-09-01-x-S_Straight_1x09_Pitch5.08mm, symbol Connector:Conn_01x09_Socket
- removed JP1: SolderJumper_2_Open, Jumper:SolderJumper-2_P1.3mm_Open_Pad1.0x1.5mm, symbol Jumper:SolderJumper_2_Open
- removed Q1: FDN340P, Package_TO_SOT_SMD:SOT-23, symbol Transistor_FET:FDN340P
- removed R1B1: 1k, Resistor_SMD:R_0603_1608Metric, symbol Device:R
- removed R3, R4: 10k, Resistor_SMD:R_0603_1608Metric, symbol Device:R
- removed U3: LP2985-3.3, Package_TO_SOT_SMD:SOT-23-5, symbol Regulator_Linear:LP2985-3.3
- removed U6: LMV358, Library:TO229P990X238-3N, symbol Amplifier_Operational:LMV358
- added BT1: 1048, Library:BAT_1048, symbol New_Library_0:1048
- added C19, C20: 10uf, Capacitor_SMD:C_0805_2012Metric_Pad1.18x1.45mm_HandSolder, symbol Device:C
- added D25: Red_Led, LED_SMD:LED_0805_2012Metric_Pad1.15x1.40mm_HandSolder, symbol Device:LED
- added D26: Green _Led, LED_SMD:LED_0805_2012Metric_Pad1.15x1.40mm_HandSolder, symbol Device:LED
- added R1A2: 2k, Resistor_SMD:R_0805_2012Metric_Pad1.20x1.40mm_HandSolder, symbol Device:R
- added R1A3, R1A4: 1k, Resistor_SMD:R_0805_2012Metric_Pad1.20x1.40mm_HandSolder, symbol Device:R
- added S1: JS202011SCQN, Library:SW_JS202011SCQN, symbol New_Library_0:JS202011SCQN
- added U10: TP4056-42-ESOP8, Library:SOIC127P600X175-9N, symbol New_Library_0:TP4056-42-ESOP8
- C5: renamed from C2; value 47u -> 10uf
- D15: renamed from D1; value D -> M7 50V 1A; footprint Diode_SMD:D_0603_1608Metric -> Diode_SMD:D_SMA
- D16: renamed from D2; value GREEN ON -> L_PWR; footprint LED_SMD:LED_0603_1608Metric -> LED_SMD:LED_0805_2012Metric_Pad1.15x1.40mm_HandSolder
- R1A1: footprint Resistor_SMD:R_0603_1608Metric -> Resistor_SMD:R_0805_2012Metric_Pad1.20x1.40mm_HandSolder
- U6: renamed from U1; footprint Package_TO_SOT_SMD:TO-252-2 -> Library:SOT229P700X180-4N
- renumbered C1 to C4, C3 to C6
Connections:
- net GND: now also BT1.N2, C19.2, C20.2, R1A2.2, U10.1 (TEMP), U10.3 (GND), U10.9 (EXP)
- net USBVCC: now also C19.1, R1A3.1, R1A4.1, U10.4 (VCC), U10.8 (CE)
- net PWRIN renamed BAT+
- net BAT+: now also S1.1, S1.4
- net VIN renamed D15_OUT
- new net: BT1.N1, BT1.P2
- new net: D26.2 (A), R1A4.2
- new net: D26.1 (K), U10.7 (~{CHRG})
- new net: D25.1 (K), U10.6 (~{STDBY})
- new net: D25.2 (A), R1A3.2
- new net: R1A2.1, U10.2 (PROG)
- new net B+: BT1.P1, C20.1, S1.2, S1.5, U10.5 (BAT)
- no-connect marks 1 -> 2
Other:
- note added: "3.7V Li-ion Battery"
- note added: "Battery Charging"
- note added: "Led Indicator Regulated Power"
- note added: "NO Thermal Proetection"
- note added: "USB_v regulator 5V"
- moved on the sheet: C4, C5, C6, D15, D16, R1A1, U6
