File: Arduino_UNO_R3/arduino_uno_r3/USB.kicad_sch (KiCad schematic)
At the start: 23 parts, among them J3 USB-B-S-X-X-TH-TR, J4 ICSP HEADER, J5 Conn_01x04_Socket, U4 ATmega16U2-M, Y1 CSTCE16M0V53-R0

Commit message: dont know updates
Parts:
- removed C6: 1u, Capacitor_SMD:C_0603_1608Metric, symbol Device:C
- removed C7: 100n, Capacitor_SMD:C_1825_4564Metric, symbol Device:C
- removed C8: 100n, Capacitor_SMD:C_0603_1608Metric, symbol Device:C
- removed D3: D, Diode_SMD:D_0603_1608Metric, symbol Device:D
- removed F1: MF-MSMF050-2, Library:FUSM1812X02, symbol New_Library_0:MF-MSMF050-2
- removed FL1: BLM21SP111SH1D, Library:BEADC2012X105N, symbol New_Library_0:BLM21SP111SH1D
- removed J3: USB-B-S-X-X-TH-TR, Library:SAMTEC_USB-B-S-X-X-TH-TR, symbol New_Library_0:USB-B-S-X-X-TH-TR
- removed J4: ICSP HEADER, Library:SAMTEC_TSS-103-03-L-D, symbol New_Library_0:ICSP HEADER
- removed J5: Conn_01x04_Socket, Connector_Samtec_HPM_THT:Samtec_HPM-04-01-x-S_Straight_1x04_Pitch5.08mm, symbol Connector:Conn_01x04_Socket
- removed JP2: SolderJumper_2_Open, TestPoint:TestPoint_2Pads_Pitch2.54mm_Drill0.8mm, symbol Jumper:SolderJumper_2_Open
- removed R10: 1M, Resistor_SMD:R_0603_1608Metric, symbol Device:R
- removed R11: 1k, Resistor_SMD:R_0603_1608Metric, symbol Device:R
- removed R5: 10k, Resistor_SMD:R_0603_1608Metric, symbol Device:R
- removed R6, R7: 22R, Resistor_SMD:R_0603_1608Metric, symbol Device:R
- removed RV1, RV2: CG0603MLC-05E, Library:VARC1608X56N, symbol New_Library_0:CG0603MLC-05E
- removed U4: ATmega16U2-M, Package_DFN_QFN:QFN-32-1EP_5x5mm_P0.5mm_EP3.1x3.1mm, symbol MCU_Microchip_ATmega:ATmega16U2-M
- removed Y1: CSTCE16M0V53-R0, Library:OSC_CSTCE16M0V53-R0, symbol New_Library_0:CSTCE16M0V53-R0
- added C11, C12, C13, C15: 0.1uf, Capacitor_SMD:C_0805_2012Metric_Pad1.18x1.45mm_HandSolder, symbol Device:C
- added C14: 10uf, Capacitor_SMD:C_0805_2012Metric_Pad1.18x1.45mm_HandSolder, symbol Device:C
- added C16: 100nf, Capacitor_SMD:C_0805_2012Metric_Pad1.18x1.45mm_HandSolder, symbol Device:C
- added D18: M7 50V 1A, Diode_SMD:D_SMA, symbol Device:D
- added J15: USB_C_Receptacle_USB2.0_16P, Connector_USB:USB_C_Receptacle_HRO_TYPE-C-31-M-12, symbol Connector:USB_C_Receptacle_USB2.0_16P
- added R35, R36: 5.1k, Resistor_SMD:R_0805_2012Metric_Pad1.20x1.40mm_HandSolder, symbol Device:R
- added U8: CH340C, Package_SO:SOIC-16_3.9x9.9mm_P1.27mm, symbol Interface_USB:CH340C
- D19: renamed from D4; footprint LED_SMD:LED_0603_1608Metric -> LED_SMD:LED_0805_2012Metric_Pad1.15x1.40mm_HandSolder
- D20: renamed from D5; footprint LED_SMD:LED_0603_1608Metric -> LED_SMD:LED_0805_2012Metric_Pad1.15x1.40mm_HandSolder
- R37: renamed from R8; value 1k -> 4.7k; footprint Resistor_SMD:R_0603_1608Metric -> Resistor_SMD:R_0805_2012Metric_Pad1.20x1.40mm_HandSolder
- R38: renamed from R9; value 1k -> 4.7k; footprint Resistor_SMD:R_0603_1608Metric -> Resistor_SMD:R_0805_2012Metric_Pad1.20x1.40mm_HandSolder
Connections:
- net RXLED is gone; now on net RXM8: D20.1 (K)
- net TXLED is gone; now on net TXM8: D19.1 (K)
- net +5V: now also U8.16 (VCC)
- net GND: now also C11.2, C12.2, C13.2, C14.2, C15.1, J15.A1 (GND), J15.A12 (GND), J15.B1 (GND), J15.B12 (GND), J15.S1 (SHIELD), R35.1, R36.1, U8.1 (GND)
- net RXM8: now also U8.2 (TXD)
- net TXM8: now also U8.3 (RXD)
- net USBVCC: now also C11.1, C12.1, C13.1, C14.1, D18.1 (K)
- new net: D18.2 (A), J15.A4 (VBUS), J15.A9 (VBUS), J15.B4 (VBUS), J15.B9 (VBUS)
- new net: J15.A5 (CC1), R35.2
- new net: J15.B5 (CC2), R36.2
- new net: C16.1, U8.13 (~{DTR})
- new net: C15.2, U8.4 (V3)
- new net D+: J15.A6 (D+), J15.B6 (D+), U8.5 (UD+)
- new net D-: J15.A7 (D-), J15.B7 (D-), U8.6 (UD-)
- new net PC6/~{RESET}: C16.2
- no-connect marks 9 -> 8
Other:
- note added: "RX_TX Indicator"
- note added: "USB Driver CH340C"
- note added: "USB_Receptacle"
- moved on the sheet: D19, D20, R37, R38
