File: BATTERY_MANAGEMENT_CIRCUIT/BATTERY_MANAGEMENT_CIRCUIT/BATTERY_MANAGEMENT_CIRCUIT.kicad_sch (KiCad schematic)
At the start: 24 parts, among them J1 OUTPUT, J2 BATTERY, J3 Conn_01x02_Socket, J4 Conn_01x02_Socket, J5 UJC-HP-3-SMT-TR, U1 IP5306

Commit message: changes and added BMC
Parts:
- added J6: TP1, TestPoint:TestPoint_2Pads_Pitch2.54mm_Drill0.8mm, symbol Connector:Screw_Terminal_01x02
- C1, C2, C4, C7: footprint Capacitor_SMD:C_0603_1608Metric -> Capacitor_THT:C_Disc_D3.0mm_W2.0mm_P2.50mm
- C3, C5, C6: footprint Capacitor_SMD:C_0603_1608Metric -> Capacitor_THT:C_Disc_D4.3mm_W1.9mm_P5.00mm
- D1, D2, D3, D4: footprint LED_SMD:LED_0805_2012Metric -> LED_THT:LED_D3.0mm
- R1, R2, R3, R4, R5, R6: footprint Resistor_SMD:R_0603_1608Metric -> Resistor_THT:R_Axial_DIN0204_L3.6mm_D1.6mm_P5.08mm_Horizontal
Connections:
- net GND: now also J6.1 (Pin_1)
- net at C1.1, R1.2: now also J6.2 (Pin_2)
Other:
- moved on the sheet: C1
Changed lines of the file:
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@@
 	(paper "A4")
 	(junction
+		(at 35.56 60.96)
+		(diameter 0)
+		(color 0 0 0 0)
+	)
+	(junction
 		(at 107.95 20.32)
 		(diameter 0)
@@
 	)
 	(junction
+		(at 34.29 50.8)
+		(diameter 0)
+		(color 0 0 0 0)
+	)
+	(junction
 		(at 135.89 44.45)
 		(diameter 0)
@@
 	)
 	(junction
-		(at 34.29 63.5)
+		(at 43.18 60.96)
 		(diameter 0)
 		(color 0 0 0 0)
@@
 	(wire
 		(pts
-			(xy 34.29 60.96) (xy 34.29 63.5)
+			(xy 43.18 58.42) (xy 43.18 60.96)
 		)
 		(stroke
@@
 	(wire
 		(pts
-			(xy 34.29 44.45) (xy 34.29 53.34)
+			(xy 93.98 64.77) (xy 106.68 64.77)
 		)
 		(stroke
@@
 	(wire
 		(pts
-			(xy 93.98 64.77) (xy 106.68 64.77)
+			(xy 27.94 55.88) (xy 27.94 60.96)
+		)
+		(stroke
+			(width 0)
+			(type default)
+		)
+	)
+	(wire
+		(pts
+			(xy 27.94 60.96) (xy 35.56 60.96)
 		)
 		(stroke
@@
 	(wire
 		(pts
-			(xy 34.29 63.5) (xy 34.29 64.77)
+			(xy 43.18 60.96) (xy 43.18 62.23)
 		)
 		(stroke
@@
 	(wire
 		(pts
+			(xy 34.29 53.34) (xy 34.29 50.8)
+		)
+		(stroke
+			(width 0)
+			(type default)
+		)
+	)
+	(wire
+		(pts
 			(xy 106.68 72.39) (xy 106.68 76.2)
 		)
@@
 	(wire
 		(pts
+			(xy 27.94 53.34) (xy 34.29 53.34)
+		)
+		(stroke
+			(width 0)
+			(type default)
+		)
+	)
+	(wire
+		(pts
 			(xy 121.92 41.91) (xy 132.08 41.91)
 		)
@@
 	(wire
 		(pts
-			(xy 26.67 63.5) (xy 34.29 63.5)
+			(xy 35.56 60.96) (xy 43.18 60.96)
 		)
 		(stroke
@@
 	(wire
 		(pts
+			(xy 43.18 50.8) (xy 34.29 50.8)
+		)
+		(stroke
+			(width 0)
+			(type default)
+		)
+	)
+	(wire
+		(pts
+			(xy 34.29 50.8) (xy 34.29 44.45)
+		)
+		(stroke
+			(width 0)
+			(type default)
+		)
+	)
+	(wire
+		(pts
 			(xy 105.41 41.91) (xy 110.49 41.91)
 		)
@@
 	(label "LED1"
 		(at 50.8 68.58 180)
+		(fields_autoplaced yes)
 		(effects
 			(font
@@
 			)
 		)
-		(property "Footprint" "Capacitor_SMD:C_0603_1608Metric"
+		(property "Footprint" "Capacitor_THT:C_Disc_D3.0mm_W2.0mm_P2.50mm"
 			(at 106.3752 49.53 0)
 			(effects
@@
 			)
 		)
-		(property "Footprint" "Capacitor_SMD:C_0603_1608Metric"
+		(property "Footprint" "Capacitor_THT:C_Disc_D4.3mm_W1.9mm_P5.00mm"
 			(at 108.9152 27.94 0)
 			(effects
@@
 			)
 		)
-		(property "Footprint" "Resistor_SMD:R_0603_1608Metric"
+		(property "Footprint" "Resistor_THT:R_Axial_DIN0204_L3.6mm_D1.6mm_P5.08mm_Horizontal"
 			(at 95.758 68.58 90)
 			(effects
@@
 			)
 		)
-		(property "Footprint" "Capacitor_SMD:C_0603_1608Metric"
+		(property "Footprint" "Capacitor_THT:C_Disc_D3.0mm_W2.0mm_P2.50mm"
 			(at 122.8852 49.53 0)
 			(effects
@@
 			)
 		)
-		(property "Footprint" "Resistor_SMD:R_0603_1608Metric"
+		(property "Footprint" "Resistor_THT:R_Axial_DIN0204_L3.6mm_D1.6mm_P5.08mm_Horizontal"
 			(at 114.3 43.688 90)
 			(effects
@@
 			)
 		)
-		(property "Footprint" "LED_SMD:LED_0805_2012Metric"
+		(property "Footprint" "LED_THT:LED_D3.0mm"
 			(at 67.31 76.2 0)
 			(effects
@@
 			)
 		)
-		(property "Footprint" "Resistor_SMD:R_0603_1608Metric"
+		(property "Footprint" "Resistor_THT:R_Axial_DIN0204_L3.6mm_D1.6mm_P5.08mm_Horizontal"
 			(at 108.458 68.58 90)
 			(effects
@@
 	)
 	(symbol
+		(lib_id "Connector:Screw_Terminal_01x02")
+		(at 22.86 55.88 180)
+		(unit 1)
+		(exclude_from_sim no)
+		(in_bom yes)
+		(on_board yes)
+		(dnp no)
+		(fields_autoplaced yes)
+		(property "Reference" "J6"
+			(at 22.86 46.99 0)
+			(effects
+				(font
+					(size 1.27 1.27)
+				)
+			)
+		)
+		(property "Value" "TP1"
+			(at 22.86 49.53 0)
+			(effects
+				(font
+					(size 1.27 1.27)
+				)
+			)
+		)
+		(property "Footprint" "TestPoint:TestPoint_2Pads_Pitch2.54mm_Drill0.8mm"
+			(at 22.86 55.88 0)
+			(effects
+				(font
+					(size 1.27 1.27)
+				)
+				(hide yes)
+			)
+		)
+		(property "Datasheet" "~"
+			(at 22.86 55.88 0)
+			(effects
+				(font
+					(size 1.27 1.27)
+				)
+				(hide yes)
+			)
+		)
+		(property "Description" "Generic screw terminal, single row, 01x02, script generated (kicad-library-utils/schlib/autogen/connector/)"
+			(at 22.86 55.88 0)
+			(effects
+				(font
+					(size 1.27 1.27)
+				)
+				(hide yes)
+			)
+		)
+		(pin "2"
+		)
+		(pin "1"
+		)
+		(instances
+			(project ""
+				(path "/331a7c19-dc29-4c39-b10d-7e761c1a62ed"
+					(reference "J6")
+					(unit 1)
+				)
+			)
+		)
+	)
+	(symbol
 		(lib_id "power:PWR_FLAG")
-		(at 26.67 63.5 0)
+		(at 35.56 60.96 0)
 		(mirror y)
 		(unit 1)
@@
 		(dnp no)
 		(property "Reference" "#FLG01"
-			(at 26.67 61.595 0)
+			(at 35.56 59.055 0)
 			(effects
 				(font
@@
 		)
 		(property "Value" "PWR_FLAG"
-			(at 26.67 58.42 0)
+			(at 35.56 55.88 0)
 			(effects
 				(font
@@
 		)
 		(property "Footprint" ""
-			(at 26.67 63.5 0)
+			(at 35.56 60.96 0)
 			(effects
 				(font
@@
 		)
 		(property "Datasheet" "~"
-			(at 26.67 63.5 0)
+			(at 35.56 60.96 0)
 			(effects
 				(font
@@
 		)
 		(property "Description" "Special symbol for telling ERC where power comes from"
-			(at 26.67 63.5 0)
+			(at 35.56 60.96 0)
 			(effects
 				(font
@@
 			)
 		)
-		(property "Footprint" "Capacitor_SMD:C_0603_1608Metric"
+		(property "Footprint" "Capacitor_THT:C_Disc_D3.0mm_W2.0mm_P2.50mm"
 			(at 50.4952 44.45 0)
 			(effects
@@
 			)
 		)
-		(property "Footprint" "Resistor_SMD:R_0603_1608Metric"
+		(property "Footprint" "Resistor_THT:R_Axial_DIN0204_L3.6mm_D1.6mm_P5.08mm_Horizontal"
 			(at 32.512 40.64 90)
 			(effects
@@
 			)
 		)
-		(property "Footprint" "LED_SMD:LED_0805_2012Metric"
+		(property "Footprint" "LED_THT:LED_D3.0mm"
 			(at 80.01 76.2 0)
 			(effects
@@
 			)
 		)
-		(property "Footprint" "Resistor_SMD:R_0603_1608Metric"
+		(property "Footprint" "Resistor_THT:R_Axial_DIN0204_L3.6mm_D1.6mm_P5.08mm_Horizontal"
 			(at 170.688 66.04 90)
 			(effects
@@
 			)
 		)
-		(property "Footprint" "Resistor_SMD:R_0603_1608Metric"
+		(property "Footprint" "Resistor_THT:R_Axial_DIN0204_L3.6mm_D1.6mm_P5.08mm_Horizontal"
 			(at 161.798 66.04 90)
 			(effects
@@
 			)
 		)
-		(property "Footprint" "Capacitor_SMD:C_0603_1608Metric"
+		(property "Footprint" "Capacitor_THT:C_Disc_D4.3mm_W1.9mm_P5.00mm"
 			(at 120.3452 27.94 0)
 			(effects
@@
 	(symbol
 		(lib_id "power:GND")
-		(at 34.29 64.77 0)
+		(at 43.18 62.23 0)
 		(unit 1)
 		(exclude_from_sim no)
@@
 		(dnp no)
 		(property "Reference" "#PWR01"
-			(at 34.29 71.12 0)
+			(at 43.18 68.58 0)
 			(effects
 				(font
@@
 		)
 		(property "Value" "GND"
-			(at 34.29 69.85 0)
+			(at 43.18 67.31 0)
 			(effects
 				(font
@@
 		)
 		(property "Footprint" ""
-			(at 34.29 64.77 0)
+			(at 43.18 62.23 0)
 			(effects
 				(font
@@
 		)
 		(property "Datasheet" ""
-			(at 34.29 64.77 0)
+			(at 43.18 62.23 0)
 			(effects
 				(font
@@
 		)
 		(property "Description" "Power symbol creates a global label with name \"GND\" , ground"
-			(at 34.29 64.77 0)
+			(at 43.18 62.23 0)
 			(effects
 				(font
@@
 			)
 		)
-		(property "Footprint" "Capacitor_SMD:C_0603_1608Metric"
+		(property "Footprint" "Capacitor_THT:C_Disc_D4.3mm_W1.9mm_P5.00mm"
 			(at 98.7552 27.94 0)
 			(effects
@@
 			)
 		)
-		(property "Footprint" "LED_SMD:LED_0805_2012Metric"
+		(property "Footprint" "LED_THT:LED_D3.0mm"
 			(at 44.45 76.2 0)
 			(effects
@@
 			)
 		)
-		(property "Footprint" "LED_SMD:LED_0805_2012Metric"
+		(property "Footprint" "LED_THT:LED_D3.0mm"
 			(at 57.15 76.2 0)
 			(effects
@@
 	(symbol
 		(lib_id "Device:C")
-		(at 34.29 57.15 0)
+		(at 43.18 54.61 0)
 		(unit 1)
 		(exclude_from_sim no)
@@
 		(fields_autoplaced yes)
 		(property "Reference" "C1"
-			(at 38.1 55.8799 0)
+			(at 46.99 53.3399 0)
 			(effects
 				(font
@@
 		)
 		(property "Value" "10uf"
-			(at 38.1 58.4199 0)
+			(at 46.99 55.8799 0)
 			(effects
 				(font
@@
 			)
 		)
-		(property "Footprint" "Capacitor_SMD:C_0603_1608Metric"
-			(at 35.2552 60.96 0)
+		(property "Footprint" "Capacitor_THT:C_Disc_D3.0mm_W2.0mm_P2.50mm"
+			(at 44.1452 58.42 0)
 			(effects
 				(font
@@
 		)
 		(property "Datasheet" "~"
-			(at 34.29 57.15 0)
+			(at 43.18 54.61 0)
 			(effects
 				(font
@@
 		)
 		(property "Description" "Unpolarized capacitor"
-			(at 34.29 57.15 0)
+			(at 43.18 54.61 0)
 			(effects
 				(font
