File: Example Project Complex/Mosfet Driver.kicad_sch (KiCad schematic)
At the start: 40 parts

Commit message: dont know updates
Parts:
- D4: renamed from D?; value D_Schottky -> PMEGA6020
- D5: renamed from D?; value D_Schottky -> BAT60A
- gave numbers to parts that had none: 38
Other:
- note added: "--->PROVIDES INSTANTANEOUS POWER TO IC DURING TRANSIENT TIME"
- note added: "BOOTSTRAP_CAP"
- note added: "DRIVE MOSFET GATE _x"
- note added: "HIGH SIDE MOSFET SOURCE_x"
- note added: "INCREASES CAPACITANCE AND REDUCED INDUCTANCE ---> IMPEDENCE DECREASE"
- note added: "KEEP AWAY FROM NOISY TRACKS AND COMPONENTS"
- note added: "SAVES ISSUE FROM +5V SUPPLY"
- note added: "SENSE 3 PHASE VOLTAGES"
- moved on the sheet: R17, R18, R19, R20, R21, R22
