File: Heart Sensor/Heart Sensor.kicad_pcb (KiCad board)
At the start: 2 copper layers, 131.1 x 44.7 mm, 18 parts, among them J1 Screw_Terminal_01x02, J3 Conn_01x02_Socket, P1 OLED 128X64 0.96, Q1 NPN, SW1 RotaryEncoder_Switch, U1 L7805, U2 MAX30100 MODULE

Commit message: dont know updates
Other:
- board text added: "HEART SENSOR PRODUCT"
Changed lines of the file:
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@@
 		(layer "Edge.Cuts")
+	)
+	(gr_text "HEART SENSOR PRODUCT"
+		(at 49.35 50.4 0)
+		(layer "F.SilkS")
+		(effects
+			(font
+				(size 2.5 2.5)
+				(thickness 0.6)
+				(bold yes)
+			)
+			(justify left bottom)
+		)
 	)
 	(segment
